Commit message: first commit

File: fw_description/urdf/fw_rev_04_jay.xacro (robot description, xacro)
@@ -13,16 +13,16 @@
     <parent link="base_footprint"/>
     <child link="base_link" />
-    <origin xyz="0 0 0.085" rpy="0 0 0"/>
+    <origin xyz="0 0 0.124" rpy="0 0 0"/>
   </joint>
   <link name="base_link">
     <visual>
-      <origin xyz="0 0 0" rpy="0 0 0"/>
-      <geometry>
-        <mesh filename="package://fw_rev_04_description/meshes/bases/newHotelRobot.stl" scale="0.001 0.001 0.001"/>
+      <origin xyz="0 0 0" rpy="0 0 ${PI/2}"/>
+      <geometry>
+        <mesh filename="package://fw_rev_04_description/meshes/freeway_hospital/base_link.STL" scale="0.001 0.001 0.001"/>
       </geometry>
       <material name="grey"/>
     </visual>
     <collision>
-      <origin xyz="0 0 0.085" rpy="0 0 0"/>
+      <origin xyz="-0.15 0 0.51" rpy="0 0 0"/>
       <geometry>
         <box size="${bodyLength} ${bodyWidth} ${bodyHeight}"/>
@@ -45,23 +45,74 @@
   </joint>
   <link name="imu_link"/> -->
-  <joint name="scan_joint" type="fixed">
-    <parent link="base_link"/>
-    <child link="base_scan"/>
-    <origin xyz="0.2423 0 0.0091" rpy="0 0 ${PI}"/>
-  </joint>
-  <link name="base_scan">
-  <visual>
-    <origin xyz="0 0 0" rpy="-${PI/2} 0 0"/>
-    <geometry>
-      <mesh filename="package://fw_rev_04_description/meshes/sensors/rplidar_s2.stl" scale="0.001 0.001 0.001"/>
+<!---->
+<!--  <joint name="scan_joint" type="fixed">-->
+<!--    <parent link="base_link"/>-->
+<!--    <child link="base_scan"/>-->
+<!--    <origin xyz="0.468 0 0.096" rpy="0 0 ${PI}"/>-->
+<!--  </joint>-->
+<!---->
+<!--  <link name="base_scan">-->
+<!--  <visual>-->
+<!--    <origin xyz="0 0 0" rpy="-${PI/2} 0 0"/>-->
+<!--    <geometry>-->
+<!--      <mesh filename="package://fw_rev_04_description/meshes/sensors/rplidar_s2.stl" scale="0.001 0.001 0.001"/>-->
+<!--    </geometry>-->
+<!--    <material name="blue"/>-->
+<!--  </visual>-->
+<!--  <collision>-->
+<!--    <origin xyz="0.015 0 -0.0065" rpy="0 0 0"/>-->
+<!--    <geometry>-->
+<!--      <cylinder length="0.0315" radius="0.055"/>-->
+<!--    </geometry>-->
+<!--  </collision>-->
+<!--  <inertial>-->
+<!--    <mass value="0.114" />-->
+<!--    <origin xyz="0 0 0" />-->
+<!--    <inertia ixx="0.001" ixy="0.0" ixz="0.0"-->
+<!--             iyy="0.001" iyz="0.0"-->
+<!--             izz="0.001" />-->
+<!--  </inertial>-->
+<!--  </link>-->
+  <joint name="scan_richbeam_joint" type="fixed">
+    <parent link="base_link"/>
+    <child link="base_scan_richbeam"/>
+    <origin xyz="0.78202 0 0.03044" rpy="0 0 0"/>
+  </joint>
+  <link name="base_scan_richbeam">
+  <visual>
+    <origin xyz="0 0 0" rpy="0 0 0"/>
+    <geometry>
+      <mesh filename="package://fw_rev_04_description/meshes/sensors/richbeam.stl" scale="0.001 0.001 0.001"/>
     </geometry>
     <material name="blue"/>
   </visual>
-  <collision>
-    <origin xyz="0.015 0 -0.0175" rpy="0 0 0"/>
-    <geometry>
-      <cylinder length="0.0315" radius="0.055"/>
-    </geometry>
-  </collision>
+  </link>
+  <joint name="scan_richbeam_joint_r" type="fixed">
+    <parent link="base_link"/>
+    <child link="base_scan_richbeam_r"/>
+    <origin xyz="0.78202 -0.25628 0.03044" rpy="0 0 -0.5236"/>
+  </joint>
+  <link name="base_scan_richbeam_r">
+  <visual>
+    <origin xyz="0 0 0" rpy="0 0 0"/>
+    <geometry>
+      <mesh filename="package://fw_rev_04_description/meshes/freeway_hospital/base_scan_right_link.STL" scale="0.001 0.001 0.001"/>
+    </geometry>
+    <material name="blue"/>
+  </visual>
+  </link>
+  <joint name="scan_richbeam_joint_l" type="fixed">
+    <parent link="base_link"/>
+    <child link="base_scan_richbeam_l"/>
+    <origin xyz="0.78202 0.25628 0.03044" rpy="0 0 0.5236"/>
+  </joint>
+  <link name="base_scan_richbeam_l">
+  <visual>
+    <origin xyz="0 0 0" rpy="0 0 0"/>
+    <geometry>
+      <mesh filename="package://fw_rev_04_description/meshes/freeway_hospital/base_scan_left_link.STL" scale="0.001 0.001 0.001"/>
+    </geometry>
+    <material name="blue"/>
+  </visual>
   </link>
   <!-- <joint name="scan_joint2" type="fixed">
@@ -236,6 +287,9 @@
     </visual>
   </link> -->
-  <xacro:sensor_d455 parent="base_link" name="d455" use_nominal_extrinsics="$(arg use_nominal_extrinsics)">
-    <origin xyz="0.2245 0 0.2225" rpy="0 0 0"/>
+  <xacro:sensor_d455 parent="base_link" name="d455_R" use_nominal_extrinsics="$(arg use_nominal_extrinsics)">
+    <origin xyz="0.74384 -0.225 0.13249" rpy="0 0 0"/>
+  </xacro:sensor_d455>
+  <xacro:sensor_d455 parent="base_link" name="d455_L" use_nominal_extrinsics="$(arg use_nominal_extrinsics)">
+    <origin xyz="0.74384 0.225 0.13249" rpy="0 0 0"/>
   </xacro:sensor_d455>
 </robot>
